Commit message: tb3_bringup: Waffle Pi URDF with front LDS-03, lidar + body filter, tb-for-rl rename
- urdf: TurtleBot3 Waffle Pi dims, top plate removed, LDS-03 on 1st floor front
- tb-only: coin_d4_driver (deps.repos) -> scan_raw -> laser_filters box -> /scan
- udev: 99-tb3-lidar.rules (/dev/tb3_lidar), install-udev installs both
- nav2 footprint polygon for Waffle Pi; wheel_separation 0.287
- fix logger.warn -> warning (Lyrical)

Co-Authored-By: Claude Opus 5.5 <noreply@anthropic.com>

File: ros2_ws/src/tb3_bringup/urdf/robot.urdf.xacro (robot description, xacro)
@@ -1,28 +1,31 @@
 <?xml version="1.0"?>
 <!--
-  TurtleBot3 Burger 개조형: 맨 위 판(라이다 자리) 걷어냄 · 라이다를 1층 앞쪽에 앞으로 조금 튀어나오게.
-  치수 출처: turtlebot3_burger.urdf (ROBOTIS, Apache 2.0) — 바퀴·캐스터·몸통 외곽은 원본 그대로.
+  TurtleBot3 Waffle Pi 개조형: 맨 위 판(원래 라이다 자리) 걷어냄 · LDS-03 라이다를 1층 앞쪽에 앞으로 조금 튀어나오게.
+  치수 출처: turtlebot3_description/urdf/turtlebot3_waffle_pi.urdf (ROBOTIS, Apache 2.0) —
+  바퀴·캐스터·몸통 외곽은 원본 그대로. 라이다 크기는 LDS-03 e-Manual (54.7 W × 39.7 D × 34 H mm).
   ★ 실측해서 고칠 값 = 아래 property 중 "측정" 표시. 바꾸면 colcon build 후 view-model로 다시 확인.
   좌표: base_link(바퀴축 높이, 바닥+0.010) — x 앞 · y 왼쪽 · z 위. 루트는 base_link
   (드라이버가 odom→base_link를 내므로 base_footprint를 위에 두면 부모가 둘이 됨 — tool·Nav2도 base_link 기준).
-  원본 몸통은 base_link 기준 x -0.102 ~ +0.038 (앞끝 0.038), z 0 ~ 0.143.
+  원본 몸통: 중심 x -0.064, 266×266mm → x -0.197 ~ +0.069 (앞끝 0.069), 높이 z 0 ~ 0.094.
 -->
-<robot name="tb3_burger_lowlidar" xmlns:xacro="http://www.ros.org/wiki/xacro">
-  <!-- 몸통 판 (Burger 와플판 140×140mm). 원본은 4층(맨 위=라이다판). 맨 위를 뺀 3층만 그림 -->
-  <xacro:property name="body_x" value="-0.032"/>          <!-- 판 중심 x (원본) -->
-  <xacro:property name="plate" value="0.140"/>
+<robot name="tb3_waffle_pi_lowlidar" xmlns:xacro="http://www.ros.org/wiki/xacro">
+  <!-- 몸통 판 (Waffle 와플판 266×266mm). 원본 3층(맨 위=라이다판) → 맨 위를 뺀 2층만 -->
+  <xacro:property name="body_x" value="-0.064"/>
+  <xacro:property name="plate" value="0.266"/>
   <xacro:property name="plate_t" value="0.003"/>
   <xacro:property name="plate_z1" value="0.000"/>          <!-- 측정: 1층 판 윗면 높이 (base_link 기준) -->
-  <xacro:property name="plate_z2" value="0.047"/>          <!-- 측정: 2층 -->
-  <xacro:property name="plate_z3" value="0.094"/>          <!-- 측정: 3층 (지금 맨 위) -->
-  <!-- 라이다 (LDS 모양). base_scan = 스캔 평면 중심 = 드라이버 frame_id -->
-  <xacro:property name="lidar_x" value="0.045"/>           <!-- 측정: 앞끝(0.038)보다 조금 앞 -->
+  <xacro:property name="plate_z2" value="0.047"/>          <!-- 측정: 2층 판 (지금 맨 위) -->
+  <!-- LDS-03 라이다. base_scan = 스캔 평면 중심 = coin_d4_driver frame_id -->
+  <xacro:property name="lidar_x" value="0.075"/>           <!-- 측정: 앞끝(0.069)보다 조금 앞 (라이다 중심) -->
   <xacro:property name="lidar_y" value="0.0"/>
-  <xacro:property name="lidar_z" value="0.030"/>           <!-- 측정: 1층 판 위 스캔 평면 높이 -->
-  <xacro:property name="lidar_yaw" value="0.0"/>           <!-- 측정: 라이다 0° 방향이 로봇 앞과 다르면 (rad) -->
+  <xacro:property name="lidar_z" value="0.022"/>           <!-- 측정: 스캔 평면 높이 (1층 판 위, 2층 판 0.047 아래) -->
+  <xacro:property name="lidar_yaw" value="0.0"/>           <!-- 측정: 라이다 0°가 로봇 앞과 다르면 (rad) -->
+  <xacro:property name="lidar_w" value="0.0547"/>
+  <xacro:property name="lidar_d" value="0.0397"/>
+  <xacro:property name="lidar_h" value="0.034"/>
   <material name="plate"><color rgba="0.35 0.35 0.35 1"/></material>
   <material name="dark"><color rgba="0.15 0.15 0.15 1"/></material>
   <material name="board"><color rgba="0.1 0.45 0.2 1"/></material>
-  <material name="lidar"><color rgba="0.8 0.2 0.1 1"/></material>
+  <material name="lidar"><color rgba="0.85 0.25 0.1 1"/></material>
   <xacro:macro name="plate_visual" params="z">
     <visual>
@@ -35,31 +38,26 @@
     <xacro:plate_visual z="${plate_z1}"/>
     <xacro:plate_visual z="${plate_z2}"/>
-    <xacro:plate_visual z="${plate_z3}"/>
-    <!-- 1층: 모터 2개 (바퀴 안쪽) -->
+    <!-- 1층: 모터 2개 (바퀴 안쪽) · 배터리 (뒤쪽) -->
     <visual>
       <origin xyz="0 0 0.023"/>
-      <geometry><box size="0.034 0.120 0.046"/></geometry>
-      <material name="dark"/>
-    </visual>
-    <!-- 2층: 배터리 / 3층: OpenCR + Pi (대략) -->
-    <visual>
-      <origin xyz="${body_x} 0 ${plate_z2 + 0.012}"/>
-      <geometry><box size="0.090 0.070 0.024"/></geometry>
+      <geometry><box size="0.034 0.250 0.046"/></geometry>
       <material name="dark"/>
     </visual>
     <visual>
-      <origin xyz="${body_x} 0 ${plate_z3 + 0.010}"/>
-      <geometry><box size="0.105 0.075 0.020"/></geometry>
+      <origin xyz="-0.110 0 0.018"/>
+      <geometry><box size="0.090 0.070 0.030"/></geometry>
+      <material name="dark"/>
+    </visual>
+    <!-- 2층: OpenCR + RPi (대략) -->
+    <visual>
+      <origin xyz="${body_x} 0 ${plate_z2 + 0.012}"/>
+      <geometry><box size="0.105 0.110 0.024"/></geometry>
       <material name="board"/>
     </visual>
-    <!-- 충돌: 몸통 상자 (맨 위 판 빠진 높이) + 앞으로 나온 라이다는 base_scan에 -->
     <collision>
-      <origin xyz="${body_x} 0 ${(plate_z3 + 0.020) / 2}"/>
-      <geometry><box size="${plate} ${plate} ${plate_z3 + 0.020}"/></geometry>
+      <origin xyz="${body_x} 0 ${(plate_z2 + 0.030) / 2}"/>
+      <geometry><box size="${plate} ${plate} ${plate_z2 + 0.030}"/></geometry>
     </collision>
-    <inertial>
-      <mass value="0.8"/>
-      <inertia ixx="2.2e-03" ixy="0" ixz="0" iyy="2.1e-03" iyz="0" izz="2.0e-03"/>
-    </inertial>
+    <!-- inertial 없음: 루트 링크 inertia는 KDL(robot_state_publisher)이 경고만 냄 — 시뮬레이션 안 하므로 생략 -->
   </link>
   <xacro:macro name="wheel" params="side y mesh">
@@ -82,13 +80,17 @@
     </link>
   </xacro:macro>
-  <xacro:wheel side="left" y="0.080" mesh="left_tire.stl"/>
-  <xacro:wheel side="right" y="-0.080" mesh="right_tire.stl"/>
-  <joint name="caster_back_joint" type="fixed">
-    <parent link="base_link"/><child link="caster_back_link"/>
-    <origin xyz="-0.081 0 -0.004" rpy="-1.5708 0 0"/>
-  </joint>
-  <link name="caster_back_link">
-    <visual><geometry><box size="0.030 0.009 0.020"/></geometry><material name="dark"/></visual>
-  </link>
+  <xacro:wheel side="left" y="0.144" mesh="left_tire.stl"/>
+  <xacro:wheel side="right" y="-0.144" mesh="right_tire.stl"/>
+  <xacro:macro name="caster" params="side y">
+    <joint name="caster_back_${side}_joint" type="fixed">
+      <parent link="base_link"/><child link="caster_back_${side}_link"/>
+      <origin xyz="-0.177 ${y} -0.004" rpy="-1.5708 0 0"/>
+    </joint>
+    <link name="caster_back_${side}_link">
+      <visual><geometry><box size="0.030 0.009 0.020"/></geometry><material name="dark"/></visual>
+    </link>
+  </xacro:macro>
+  <xacro:caster side="left" y="0.064"/>
+  <xacro:caster side="right" y="-0.064"/>
   <joint name="scan_joint" type="fixed">
     <parent link="base_link"/><child link="base_scan"/>
@@ -96,12 +98,11 @@
   </joint>
   <link name="base_scan">
+    <!-- LDS-03 외형 (상자로 근사, 스캔 평면이 높이 중앙이라고 가정) -->
     <visual>
-      <!-- lds.stl 원점 = 스캔 중심 (원본 TB3와 같음) -->
-      <geometry><mesh filename="package://tb3_bringup/meshes/lds.stl" scale="0.001 0.001 0.001"/></geometry>
+      <geometry><box size="${lidar_d} ${lidar_w} ${lidar_h}"/></geometry>
       <material name="lidar"/>
     </visual>
     <collision>
-      <origin xyz="0.015 0 -0.0065"/>
-      <geometry><cylinder length="0.0315" radius="0.055"/></geometry>
+      <geometry><box size="${lidar_d} ${lidar_w} ${lidar_h}"/></geometry>
     </collision>
   </link>

Commit message: urdf: LDS-03 between front wheels, OpenCR front / RPi back on 2nd plate (from photo)
Co-Authored-By: Claude Opus 5.5 <noreply@anthropic.com>

File: ros2_ws/src/tb3_bringup/urdf/robot.urdf.xacro (robot description, xacro)
@@ -1,5 +1,6 @@
 <?xml version="1.0"?>
 <!--
-  TurtleBot3 Waffle Pi 개조형: 맨 위 판(원래 라이다 자리) 걷어냄 · LDS-03 라이다를 1층 앞쪽에 앞으로 조금 튀어나오게.
+  TurtleBot3 Waffle Pi 개조형: 맨 위 판(원래 라이다 자리) 걷어냄 · LDS-03 라이다를 1층 맨 앞, 두 바퀴 사이 가운데에.
+  2층(지금 맨 위): 앞쪽 OpenCR · 뒤쪽 Raspberry Pi 4 (2026-10-27 사진 기준).
   치수 출처: turtlebot3_description/urdf/turtlebot3_waffle_pi.urdf (ROBOTIS, Apache 2.0) —
   바퀴·캐스터·몸통 외곽은 원본 그대로. 라이다 크기는 LDS-03 e-Manual (54.7 W × 39.7 D × 34 H mm).
@@ -17,5 +18,5 @@
   <xacro:property name="plate_z2" value="0.047"/>          <!-- 측정: 2층 판 (지금 맨 위) -->
   <!-- LDS-03 라이다. base_scan = 스캔 평면 중심 = coin_d4_driver frame_id -->
-  <xacro:property name="lidar_x" value="0.075"/>           <!-- 측정: 앞끝(0.069)보다 조금 앞 (라이다 중심) -->
+  <xacro:property name="lidar_x" value="0.060"/>           <!-- 측정: 라이다 중심 — 바퀴축(0)보다 앞, 판 앞끝(0.069) 근처 -->
   <xacro:property name="lidar_y" value="0.0"/>
   <xacro:property name="lidar_z" value="0.022"/>           <!-- 측정: 스캔 평면 높이 (1층 판 위, 2층 판 0.047 아래) -->
@@ -49,8 +50,13 @@
       <material name="dark"/>
     </visual>
-    <!-- 2층: OpenCR + RPi (대략) -->
+    <!-- 2층: 앞쪽 OpenCR (105×75mm) · 뒤쪽 Raspberry Pi 4 (85×56mm) — 사진 기준 대략 위치 -->
     <visual>
-      <origin xyz="${body_x} 0 ${plate_z2 + 0.012}"/>
-      <geometry><box size="0.105 0.110 0.024"/></geometry>
+      <origin xyz="-0.025 0 ${plate_z2 + 0.010}"/>
+      <geometry><box size="0.075 0.105 0.020"/></geometry>
+      <material name="board"/>
+    </visual>
+    <visual>
+      <origin xyz="-0.140 -0.010 ${plate_z2 + 0.010}"/>
+      <geometry><box size="0.056 0.085 0.020"/></geometry>
       <material name="board"/>
     </visual>

Commit message: frames: REP-105 odom->base_footprint->base_link (driver, URDF, mock, SLAM, amcl)
Co-Authored-By: Claude Opus 5.5 <noreply@anthropic.com>

File: ros2_ws/src/tb3_bringup/urdf/robot.urdf.xacro (robot description, xacro)
@@ -6,6 +6,6 @@
   바퀴·캐스터·몸통 외곽은 원본 그대로. 라이다 크기는 LDS-03 e-Manual (54.7 W × 39.7 D × 34 H mm).
   ★ 실측해서 고칠 값 = 아래 property 중 "측정" 표시. 바꾸면 colcon build 후 view-model로 다시 확인.
-  좌표: base_link(바퀴축 높이, 바닥+0.010) — x 앞 · y 왼쪽 · z 위. 루트는 base_link
-  (드라이버가 odom→base_link를 내므로 base_footprint를 위에 두면 부모가 둘이 됨 — tool·Nav2도 base_link 기준).
+  좌표 (REP-105, 원본 TB3와 같음): base_footprint(바닥, 루트) → base_link(바퀴축, +0.010) — x 앞 · y 왼쪽 · z 위.
+  드라이버가 odom→base_footprint를 낸다. 아래 값은 전부 base_link 기준.
   원본 몸통: 중심 x -0.064, 266×266mm → x -0.197 ~ +0.069 (앞끝 0.069), 높이 z 0 ~ 0.094.
 -->
@@ -36,4 +36,9 @@
     </visual>
   </xacro:macro>
+  <link name="base_footprint"/>
+  <joint name="base_joint" type="fixed">
+    <parent link="base_footprint"/><child link="base_link"/>
+    <origin xyz="0 0 0.010"/>
+  </joint>
   <link name="base_link">
     <xacro:plate_visual z="${plate_z1}"/>
@@ -65,5 +70,4 @@
       <geometry><box size="${plate} ${plate} ${plate_z2 + 0.030}"/></geometry>
     </collision>
-    <!-- inertial 없음: 루트 링크 inertia는 KDL(robot_state_publisher)이 경고만 냄 — 시뮬레이션 안 하므로 생략 -->
   </link>
   <xacro:macro name="wheel" params="side y mesh">

Commit message: imu: firmware I line (OpenCR on-board gyro/accel/quat, gyro bias at boot), driver publishes /imu (imu_link), URDF imu_link
Co-Authored-By: Claude Opus 5.5 <noreply@anthropic.com>

File: ros2_ws/src/tb3_bringup/urdf/robot.urdf.xacro (robot description, xacro)
@@ -107,4 +107,10 @@
     <origin xyz="${lidar_x} ${lidar_y} ${lidar_z}" rpy="0 0 ${lidar_yaw}"/>
   </joint>
+  <!-- OpenCR 내장 IMU (보드 위치 = 위 OpenCR 상자, 축은 base_link와 같다고 가정 — 왼쪽 회전에 gz > 0 확인) -->
+  <joint name="imu_joint" type="fixed">
+    <parent link="base_link"/><child link="imu_link"/>
+    <origin xyz="-0.025 0 ${plate_z2 + 0.010}"/>
+  </joint>
+  <link name="imu_link"/>
   <link name="base_scan">
     <!-- LDS-03 외형 (상자로 근사, 스캔 평면이 높이 중앙이라고 가정) -->

Commit message: isaac v2: rl_correct on our Waffle Pi URDF, observable-only (encoder + gyro), 20 Hz, motor lag/asymmetry/deadband, WiFi latency, step commands
- robot_spec.py: one place for limits/rates; URDF -> USD
- fixes found by physics smoke: caster collision + zero friction (body was dragging), Lab 6.1 quats are xyzw (v1 had wrong yaw/reset)
- ONNX outputs physical correction (scale baked in); shared export for train/export
- zero command -> zero correction (no creep)
- remove beebot assets, nav2_rl task, debug scripts

Co-Authored-By: Claude Opus 5.5 <noreply@anthropic.com>

File: ros2_ws/src/tb3_bringup/urdf/robot.urdf.xacro (robot description, xacro)
@@ -70,4 +70,10 @@
       <geometry><box size="${plate} ${plate} ${plate_z2 + 0.030}"/></geometry>
     </collision>
+    <!-- 근사: Waffle Pi 1.8 kg에서 위판 뺀 몸체 (배터리·모터·보드·라이다). Isaac 학습용 — 바꾸면 isaac 재학습 -->
+    <inertial>
+      <origin xyz="${body_x} 0 0.030"/>
+      <mass value="1.4"/>
+      <inertia ixx="0.0090" ixy="0" ixz="0" iyy="0.0090" iyz="0" izz="0.0165"/>
+    </inertial>
   </link>
   <xacro:macro name="wheel" params="side y mesh">
@@ -99,4 +105,10 @@
     <link name="caster_back_${side}_link">
       <visual><geometry><box size="0.030 0.009 0.020"/></geometry><material name="dark"/></visual>
+      <!-- 볼 캐스터 접지점 (링크가 x축 -90° 돌아 있어 base z +0.004 = 링크 y -0.004). 반지름 0.010 → 바닥에 닿음.
+           Isaac은 이 충돌체에 마찰 0을 붙인다 (볼이 굴러감). 없으면 무게중심이 축 뒤라 몸통이 끌림. -->
+      <collision>
+        <origin xyz="0 -0.004 0"/>
+        <geometry><sphere radius="0.010"/></geometry>
+      </collision>
     </link>
   </xacro:macro>

Commit message: urdf: our robot from beebot CAD — manipulator, top plate (3rd floor) and everything on it, rear pole + camera removed; standoffs kept; LDS-03 at 1st floor front
- isaac/urdf/beebot restored as the CAD source + make_tb3_body.py (splits base_link.stl into pieces, rule-based keep)
- tb3_bringup/meshes: body.stl (3.5 MB), wheel_left/right.stl; old tire meshes removed
- wheels/casters/IMU positions from beebot CAD (IMU 0.0178, 0, 0.0585)
- checked: check_urdf, render (side/front/top), Isaac load + physics smoke (0.200 m/s, 0.996 rad/s)

Co-Authored-By: Claude Opus 5.5 <noreply@anthropic.com>

File: ros2_ws/src/tb3_bringup/urdf/robot.urdf.xacro (robot description, xacro)
@@ -1,39 +1,25 @@
 <?xml version="1.0"?>
 <!--
-  TurtleBot3 Waffle Pi 개조형: 맨 위 판(원래 라이다 자리) 걷어냄 · LDS-03 라이다를 1층 맨 앞, 두 바퀴 사이 가운데에.
-  2층(지금 맨 위): 앞쪽 OpenCR · 뒤쪽 Raspberry Pi 4 (2026-10-27 사진 기준).
-  치수 출처: turtlebot3_description/urdf/turtlebot3_waffle_pi.urdf (ROBOTIS, Apache 2.0) —
-  바퀴·캐스터·몸통 외곽은 원본 그대로. 라이다 크기는 LDS-03 e-Manual (54.7 W × 39.7 D × 34 H mm).
+  TurtleBot3 Waffle Pi 개조형 = beebot CAD(isaac/urdf/beebot)에서 매니퓰레이터 · 맨 위 판(3층)과 그 위 · 뒤 pole·카메라를 뺀 것
+  + LDS-03 라이다를 1층 맨 앞, 두 바퀴 사이 가운데에.
+  2층(지금 맨 위): 앞쪽 OpenCR · 뒤쪽 Raspberry Pi 4 · 모서리 지지봉(standoff)은 그대로 위로 솟아 있음 (2026-10-27 사진).
+  메시: meshes/body.stl · wheel_*.stl ← isaac/urdf/beebot/make_tb3_body.py가 beebot 메시에서 만듦 (mm, scale 0.001).
   ★ 실측해서 고칠 값 = 아래 property 중 "측정" 표시. 바꾸면 colcon build 후 view-model로 다시 확인.
-  좌표 (REP-105, 원본 TB3와 같음): base_footprint(바닥, 루트) → base_link(바퀴축, +0.010) — x 앞 · y 왼쪽 · z 위.
+  좌표 (REP-105): base_footprint(바닥, 루트) → base_link(바퀴축 아래, +0.010) — x 앞 · y 왼쪽 · z 위.
   드라이버가 odom→base_footprint를 낸다. 아래 값은 전부 base_link 기준.
-  원본 몸통: 중심 x -0.064, 266×266mm → x -0.197 ~ +0.069 (앞끝 0.069), 높이 z 0 ~ 0.094.
+  몸통 외곽: x -0.197 ~ +0.069 (앞끝 0.069) · y ±0.139 · z -0.010(캐스터) ~ 0.091(지지봉 끝).
 -->
 <robot name="tb3_waffle_pi_lowlidar" xmlns:xacro="http://www.ros.org/wiki/xacro">
-  <!-- 몸통 판 (Waffle 와플판 266×266mm). 원본 3층(맨 위=라이다판) → 맨 위를 뺀 2층만 -->
-  <xacro:property name="body_x" value="-0.064"/>
-  <xacro:property name="plate" value="0.266"/>
-  <xacro:property name="plate_t" value="0.003"/>
-  <xacro:property name="plate_z1" value="0.000"/>          <!-- 측정: 1층 판 윗면 높이 (base_link 기준) -->
-  <xacro:property name="plate_z2" value="0.047"/>          <!-- 측정: 2층 판 (지금 맨 위) -->
   <!-- LDS-03 라이다. base_scan = 스캔 평면 중심 = coin_d4_driver frame_id -->
   <xacro:property name="lidar_x" value="0.060"/>           <!-- 측정: 라이다 중심 — 바퀴축(0)보다 앞, 판 앞끝(0.069) 근처 -->
   <xacro:property name="lidar_y" value="0.0"/>
-  <xacro:property name="lidar_z" value="0.022"/>           <!-- 측정: 스캔 평면 높이 (1층 판 위, 2층 판 0.047 아래) -->
+  <xacro:property name="lidar_z" value="0.022"/>           <!-- 측정: 스캔 평면 높이 (1층 판 위, 2층 판 아래) -->
   <xacro:property name="lidar_yaw" value="0.0"/>           <!-- 측정: 라이다 0°가 로봇 앞과 다르면 (rad) -->
-  <xacro:property name="lidar_w" value="0.0547"/>
+  <xacro:property name="lidar_w" value="0.0547"/>          <!-- LDS-03 e-Manual 54.7 W × 39.7 D × 34 H mm -->
   <xacro:property name="lidar_d" value="0.0397"/>
   <xacro:property name="lidar_h" value="0.034"/>
-  <material name="plate"><color rgba="0.35 0.35 0.35 1"/></material>
-  <material name="dark"><color rgba="0.15 0.15 0.15 1"/></material>
-  <material name="board"><color rgba="0.1 0.45 0.2 1"/></material>
+  <material name="body"><color rgba="0.25 0.25 0.25 1"/></material>
+  <material name="dark"><color rgba="0.12 0.12 0.12 1"/></material>
   <material name="lidar"><color rgba="0.85 0.25 0.1 1"/></material>
-  <xacro:macro name="plate_visual" params="z">
-    <visual>
-      <origin xyz="${body_x} 0 ${z - plate_t / 2}"/>
-      <geometry><box size="${plate} ${plate} ${plate_t}"/></geometry>
-      <material name="plate"/>
-    </visual>
-  </xacro:macro>
   <link name="base_footprint"/>
   <joint name="base_joint" type="fixed">
@@ -42,87 +28,66 @@
   </joint>
   <link name="base_link">
-    <xacro:plate_visual z="${plate_z1}"/>
-    <xacro:plate_visual z="${plate_z2}"/>
-    <!-- 1층: 모터 2개 (바퀴 안쪽) · 배터리 (뒤쪽) -->
     <visual>
-      <origin xyz="0 0 0.023"/>
-      <geometry><box size="0.034 0.250 0.046"/></geometry>
-      <material name="dark"/>
+      <geometry><mesh filename="package://tb3_bringup/meshes/body.stl" scale="0.001 0.001 0.001"/></geometry>
+      <material name="body"/>
     </visual>
-    <visual>
-      <origin xyz="-0.110 0 0.018"/>
-      <geometry><box size="0.090 0.070 0.030"/></geometry>
-      <material name="dark"/>
-    </visual>
-    <!-- 2층: 앞쪽 OpenCR (105×75mm) · 뒤쪽 Raspberry Pi 4 (85×56mm) — 사진 기준 대략 위치 -->
-    <visual>
-      <origin xyz="-0.025 0 ${plate_z2 + 0.010}"/>
-      <geometry><box size="0.075 0.105 0.020"/></geometry>
-      <material name="board"/>
-    </visual>
-    <visual>
-      <origin xyz="-0.140 -0.010 ${plate_z2 + 0.010}"/>
-      <geometry><box size="0.056 0.085 0.020"/></geometry>
-      <material name="board"/>
-    </visual>
+    <!-- 1층~2층 + 지지봉 (판 266×266mm, 중심 x -0.064) -->
     <collision>
-      <origin xyz="${body_x} 0 ${(plate_z2 + 0.030) / 2}"/>
-      <geometry><box size="${plate} ${plate} ${plate_z2 + 0.030}"/></geometry>
+      <origin xyz="-0.064 0 0.0455"/>
+      <geometry><box size="0.266 0.266 0.091"/></geometry>
     </collision>
     <!-- 근사: Waffle Pi 1.8 kg에서 위판 뺀 몸체 (배터리·모터·보드·라이다). Isaac 학습용 — 바꾸면 isaac 재학습 -->
     <inertial>
-      <origin xyz="${body_x} 0 0.030"/>
+      <origin xyz="-0.064 0 0.030"/>
       <mass value="1.4"/>
       <inertia ixx="0.0090" ixy="0" ixz="0" iyy="0.0090" iyz="0" izz="0.0165"/>
     </inertial>
   </link>
-  <xacro:macro name="wheel" params="side y mesh">
+  <!-- 바퀴 (beebot CAD 위치·메시). +회전 = 앞으로 -->
+  <xacro:macro name="wheel" params="side y">
     <joint name="wheel_${side}_joint" type="continuous">
       <parent link="base_link"/><child link="wheel_${side}_link"/>
-      <origin xyz="0 ${y} 0.023" rpy="-1.5708 0 0"/>
-      <axis xyz="0 0 1"/>
+      <origin xyz="0 ${y} 0.023"/>
+      <axis xyz="0 1 0"/>
     </joint>
     <link name="wheel_${side}_link">
       <visual>
-        <origin rpy="1.5708 0 0"/>
-        <geometry><mesh filename="package://tb3_bringup/meshes/${mesh}" scale="0.001 0.001 0.001"/></geometry>
+        <geometry><mesh filename="package://tb3_bringup/meshes/wheel_${side}.stl" scale="0.001 0.001 0.001"/></geometry>
         <material name="dark"/>
       </visual>
-      <collision><geometry><cylinder length="0.018" radius="0.033"/></geometry></collision>
+      <collision>
+        <origin rpy="1.5708 0 0"/>
+        <geometry><cylinder length="0.015" radius="0.033"/></geometry>
+      </collision>
       <inertial>
         <mass value="0.0285"/>
-        <inertia ixx="1.1e-05" ixy="0" ixz="0" iyy="1.1e-05" iyz="0" izz="2.1e-05"/>
+        <inertia ixx="1.1e-05" ixy="0" ixz="0" iyy="2.05e-05" iyz="0" izz="1.1e-05"/>
       </inertial>
     </link>
   </xacro:macro>
-  <xacro:wheel side="left" y="0.144" mesh="left_tire.stl"/>
-  <xacro:wheel side="right" y="-0.144" mesh="right_tire.stl"/>
+  <xacro:wheel side="left" y="0.1439"/>
+  <xacro:wheel side="right" y="-0.1439"/>
+  <!-- 볼 캐스터 (모양은 body.stl에 있음 · 여기는 접지 구만). Isaac은 'caster' 충돌체에 마찰 0을 붙인다 (볼이 굴러감) -->
   <xacro:macro name="caster" params="side y">
     <joint name="caster_back_${side}_joint" type="fixed">
       <parent link="base_link"/><child link="caster_back_${side}_link"/>
-      <origin xyz="-0.177 ${y} -0.004" rpy="-1.5708 0 0"/>
+      <origin xyz="-0.177 ${y} -0.005237"/>
     </joint>
     <link name="caster_back_${side}_link">
-      <visual><geometry><box size="0.030 0.009 0.020"/></geometry><material name="dark"/></visual>
-      <!-- 볼 캐스터 접지점 (링크가 x축 -90° 돌아 있어 base z +0.004 = 링크 y -0.004). 반지름 0.010 → 바닥에 닿음.
-           Isaac은 이 충돌체에 마찰 0을 붙인다 (볼이 굴러감). 없으면 무게중심이 축 뒤라 몸통이 끌림. -->
-      <collision>
-        <origin xyz="0 -0.004 0"/>
-        <geometry><sphere radius="0.010"/></geometry>
-      </collision>
+      <collision><geometry><sphere radius="0.004763"/></geometry></collision>
     </link>
   </xacro:macro>
   <xacro:caster side="left" y="0.064"/>
   <xacro:caster side="right" y="-0.064"/>
+  <!-- OpenCR 내장 IMU (beebot 실측: 보드 윗면). 축은 base_link와 같다고 가정 — 왼쪽 회전에 gz > 0 확인 -->
+  <joint name="imu_joint" type="fixed">
+    <parent link="base_link"/><child link="imu_link"/>
+    <origin xyz="0.0178 0 0.0585"/>
+  </joint>
+  <link name="imu_link"/>
   <joint name="scan_joint" type="fixed">
     <parent link="base_link"/><child link="base_scan"/>
     <origin xyz="${lidar_x} ${lidar_y} ${lidar_z}" rpy="0 0 ${lidar_yaw}"/>
   </joint>
-  <!-- OpenCR 내장 IMU (보드 위치 = 위 OpenCR 상자, 축은 base_link와 같다고 가정 — 왼쪽 회전에 gz > 0 확인) -->
-  <joint name="imu_joint" type="fixed">
-    <parent link="base_link"/><child link="imu_link"/>
-    <origin xyz="-0.025 0 ${plate_z2 + 0.010}"/>
-  </joint>
-  <link name="imu_link"/>
   <link name="base_scan">
     <!-- LDS-03 외형 (상자로 근사, 스캔 평면이 높이 중앙이라고 가정) -->
