Commit message: isaac/urdf/beebot: now our robot — manipulator, cameras, basket, top plate and rear pole removed (standoffs kept), LDS-03 at 1st floor front; ros2_control wheels+imu only; body.stl mesh; beebot.urdf regenerated
checked: check_urdf, render from URDF, Isaac load (2 wheel joints, stands at 0.010, 1.53 kg)

Co-Authored-By: Claude Opus 5.5 <noreply@anthropic.com>

File: isaac/urdf/beebot/beebot.urdf (robot description, URDF)
Before this commit: robot beebot, 30 links, 29 joints
Links:
- removed link arm_base_link
- removed link basket_slot_0
- removed link basket_slot_1
- removed link basket_slot_10
- removed link basket_slot_11
- removed link basket_slot_2
- removed link basket_slot_3
- removed link basket_slot_4
- removed link basket_slot_5
- removed link basket_slot_6
- removed link basket_slot_7
- removed link basket_slot_8
- removed link basket_slot_9
- removed link end_effector_link
- removed link finger_left_link
- removed link finger_right_link
- removed link forearm_link
- removed link gripper_cam_color_optical_frame
- removed link gripper_cam_link
- removed link gripper_link
- removed link pole_front_cam_color_optical_frame
- removed link pole_front_cam_link
- removed link shoulder_link
- removed link upper_arm_link
- removed link wrist_link
- added link base_scan; collision box size=0.0397 0.0547 0.034; visual box size=0.0397 0.0547 0.034
- link base_link: mass 2.400600 -> 1.4; geometry collision box size=0.266000 0.266000 0.091000; collision sphere radius=0.004763
Joints:
- removed joint arm_mount_joint
- removed joint basket_slot_0_joint
- removed joint basket_slot_10_joint
- removed joint basket_slot_11_joint
- removed joint basket_slot_1_joint
- removed joint basket_slot_2_joint
- removed joint basket_slot_3_joint
- removed joint basket_slot_4_joint
- removed joint basket_slot_5_joint
- removed joint basket_slot_6_joint
- removed joint basket_slot_7_joint
- removed joint basket_slot_8_joint
- removed joint basket_slot_9_joint
- removed joint end_effector_joint
- removed joint gripper_cam_joint
- removed joint gripper_cam_optical_joint
- removed joint gripper_left_joint
- removed joint gripper_right_joint
- removed joint joint1
- removed joint joint2
- removed joint joint3
- removed joint joint4
- removed joint joint5
- removed joint pole_front_cam_joint
- removed joint pole_front_cam_optical_joint
- added joint scan_joint: type fixed, parent base_link, child base_scan, origin xyz=0.060 0 0.022 rpy=0 0 0

File: isaac/urdf/beebot/urdf.xacro (robot description, xacro)
@@ -1,559 +1,134 @@
 <?xml version="1.0" ?>
 <!--
-  beebot — 실측 CAD(bee.urdf, SolidWorks 내보내기)에서 만든 모델. bee.urdf를 새로 받으면 이 파일을 다시 만든다:
-    · 메시 경로: meshes/x.stl → meshes/x.stl
-    · 이름 맞춤(제어·시뮬레이터가 쓰는 이름): camera_rear → pole_front_cam, camera_wrist → gripper_cam,
-      gripper_joint → gripper_left_joint, gripper_mimic_joint → gripper_right_joint, tcp → end_effector
-    · 추가: imu_link · <ros2_control> 블록(BeebotSystemHardware) · xacro 인자
-  설계: documents/project/ros/07-tf.md (TF 트리), 08-ctrl.md (ros2_control)
-  좌표: base_footprint(바닥) → base_link(바퀴 축 아래 0.010m), x 앞 · y 왼쪽 · z 위
-  구동 관절 6개: joint1~5 (팔) · gripper_left_joint (평행 그리퍼, 0=닫힘 · 0.0265=열림, 오른쪽은 mimic) + 바퀴 2개
-  xacro 인자:
-    mock_hardware (false)  true면 control/BeebotSystemHardware가 실기 대신 명령을 그대로 상태로 되돌려 줌 (테스트베드)
-    mock_effort   (0.0)    mock일 때 팔 관절 effort[A] (arm_safety_monitor 시험용)
-    port          (/dev/opencr)  OpenCR 포트 (udev 고정 이름 — ros2_ws/99-opencr.rules)
+  우리 로봇 (TurtleBot3 Waffle Pi 개조) — beebot CAD(visualkhh/Lv2_bee_Assignment)에서:
+    매니퓰레이터(팔·그리퍼·손목 카메라) · 맨 위 판(3층)과 그 위(바구니·팔 받침) · 뒤 pole + 카메라 제거, 지지봉(standoff) 유지,
+    LDS-03 라이다를 1층 맨 앞에 추가. 몸통 메시 body.stl = make_tb3_body.py가 base_link.stl에서 위 부분을 뺀 것.
+  같은 로봇: ros2_ws/src/tb3_bringup/urdf/robot.urdf.xacro (ROS·Isaac 학습이 실제로 쓰는 쪽) — 값을 바꾸면 둘 다.
+  좌표: base_footprint(바닥) → base_link(바퀴 축 아래 0.010m), x 앞 · y 왼쪽 · z 위.
+  xacro 인자: mock_hardware · mock_effort · port (ros2_control, 바퀴만) · mesh_uri (메시 폴더)
+  beebot.urdf = xacro urdf.xacro mesh_uri:=meshes
 -->
-<!-- generated by make_xacro.py -->
-<robot name="beebot" xmlns:xacro="http://www.ros.org/wiki/xacro">
-  <xacro:arg name="mock_hardware" default="false"/>
-  <xacro:arg name="mock_effort" default="0.0"/>
-  <xacro:arg name="port" default="/dev/opencr"/>
-  <xacro:arg name="mesh_uri" default="package://ros_system/urdf/meshes"/>
-  <link name="base_footprint"/>
+<robot xmlns:xacro="http://www.ros.org/wiki/xacro" name="tb3_waffle_pi_lowlidar">
+  <xacro:arg name="mock_hardware" default="false" />
+  <xacro:arg name="mock_effort" default="0.0" />
+  <xacro:arg name="port" default="/dev/opencr" />
+  <xacro:arg name="mesh_uri" default="package://ros_system/urdf/meshes" />
+  <link name="base_footprint" />
   <joint name="base_joint" type="fixed">
-    <parent link="base_footprint"/>
-    <child link="base_link"/>
-    <origin rpy="0.000000 -0.000000 0.000000" xyz="0.000000 0.000000 0.010000"/>
+    <parent link="base_footprint" />
+    <child link="base_link" />
+    <origin rpy="0.000000 -0.000000 0.000000" xyz="0.000000 0.000000 0.010000" />
   </joint>
   <link name="base_link">
     <inertial>
-      <origin rpy="0 0 0" xyz="-0.050770 -0.000171 0.080461"/>  <!-- x: real balance pose 2026-10-28 (was -0.085426 from build.py) -->
-      <mass value="2.400600"/>
-      <inertia ixx="2.8130e-02" ixy="-2.1613e-05" ixz="6.4439e-03" iyy="3.2644e-02" iyz="-1.4858e-06" izz="2.7766e-02"/>
+      <!-- 근사: Waffle Pi 1.8 kg에서 위판 뺀 몸체 (팔·pole 없음). tb3_bringup URDF와 같은 값 -->
+      <origin rpy="0 0 0" xyz="-0.064 0 0.030" />
+      <mass value="1.4" />
+      <inertia ixx="0.0090" ixy="0" ixz="0" iyy="0.0090" iyz="0" izz="0.0165" />
     </inertial>
     <visual>
-      <origin rpy="0 0 0" xyz="0 0 0"/>
+      <origin rpy="0 0 0" xyz="0 0 0" />
       <geometry>
-        <mesh filename="$(arg mesh_uri)/base_link.stl" scale="0.001 0.001 0.001"/>
+        <mesh filename="$(arg mesh_uri)/body.stl" scale="0.001 0.001 0.001" />
       </geometry>
     </visual>
     <collision>
-      <origin rpy="0.000000 0.000000 0.000000" xyz="-0.081850 0.000000 0.045500"/>
+      <origin rpy="0.000000 0.000000 0.000000" xyz="-0.064000 0.000000 0.045500" />
       <geometry>
-        <box size="0.301300 0.265600 0.091000"/>
+        <box size="0.266000 0.266000 0.091000" />
       </geometry>
     </collision>
     <collision>
-      <origin rpy="0.000000 0.000000 0.000000" xyz="0.032000 0.000000 0.108675"/>
+      <origin rpy="0 0 0" xyz="-0.177000 0.064000 -0.005237" />
       <geometry>
-        <box size="0.073600 0.137600 0.035350"/>
+        <sphere radius="0.004763" />
       </geometry>
     </collision>
     <collision>
-      <origin rpy="0.000000 0.000000 0.000000" xyz="-0.209400 0.000000 0.108675"/>
+      <origin rpy="0 0 0" xyz="-0.177000 -0.064000 -0.005237" />
       <geometry>
-        <box size="0.020000 0.020000 0.035350"/>
-      </geometry>
-    </collision>
-    <collision>
-      <origin rpy="0.000000 0.000000 0.000000" xyz="0.032000 0.000000 0.131250"/>
-      <geometry>
-        <box size="0.073600 0.137600 0.009800"/>
-      </geometry>
-    </collision>
-    <collision>
-      <origin rpy="0.000000 0.000000 0.000000" xyz="-0.209400 0.000000 0.291900"/>
-      <geometry>
-        <box size="0.020000 0.020000 0.331100"/>
-      </geometry>
-    </collision>
-    <collision>
-      <origin rpy="0 0 0" xyz="-0.177000 0.064000 -0.005237"/>
-      <geometry>
-        <sphere radius="0.004763"/>
-      </geometry>
-    </collision>
-    <collision>
-      <origin rpy="0 0 0" xyz="-0.177000 -0.064000 -0.005237"/>
-      <geometry>
-        <sphere radius="0.004763"/>
-      </geometry>
-    </collision>
-    <collision name="storage_collision_0">
-      <origin rpy="1.570796 0.000000 0.000000" xyz="-0.064000 0.000000 -0.000500"/>
-      <geometry>
-        <mesh filename="$(arg mesh_uri)/storage_collision/storage_0.stl" scale="0.001 0.001 0.001"/>
-      </geometry>
-    </collision>
-    <collision name="storage_collision_1">
-      <origin rpy="1.570796 0.000000 0.000000" xyz="-0.064000 0.000000 -0.000500"/>
-      <geometry>
-        <mesh filename="$(arg mesh_uri)/storage_collision/storage_1.stl" scale="0.001 0.001 0.001"/>
-      </geometry>
-    </collision>
-    <collision name="storage_collision_2">
-      <origin rpy="1.570796 0.000000 0.000000" xyz="-0.064000 0.000000 -0.000500"/>
-      <geometry>
-        <mesh filename="$(arg mesh_uri)/storage_collision/storage_2.stl" scale="0.001 0.001 0.001"/>
-      </geometry>
-    </collision>
-    <collision name="storage_collision_3">
-      <origin rpy="1.570796 0.000000 0.000000" xyz="-0.064000 0.000000 -0.000500"/>
-      <geometry>
-        <mesh filename="$(arg mesh_uri)/storage_collision/storage_3.stl" scale="0.001 0.001 0.001"/>
-      </geometry>
-    </collision>
-    <collision name="storage_collision_4">
-      <origin rpy="1.570796 0.000000 0.000000" xyz="-0.064000 0.000000 -0.000500"/>
-      <geometry>
-        <mesh filename="$(arg mesh_uri)/storage_collision/storage_4.stl" scale="0.001 0.001 0.001"/>
-      </geometry>
-    </collision>
-    <collision name="storage_collision_5">
-      <origin rpy="1.570796 0.000000 0.000000" xyz="-0.064000 0.000000 -0.000500"/>
-      <geometry>
-        <mesh filename="$(arg mesh_uri)/storage_collision/storage_5.stl" scale="0.001 0.001 0.001"/>
-      </geometry>
-    </collision>
-    <collision name="storage_collision_6">
-      <origin rpy="1.570796 0.000000 0.000000" xyz="-0.064000 0.000000 -0.000500"/>
-      <geometry>
-        <mesh filename="$(arg mesh_uri)/storage_collision/storage_6.stl" scale="0.001 0.001 0.001"/>
-      </geometry>
-    </collision>
-    <collision name="storage_collision_7">
-      <origin rpy="1.570796 0.000000 0.000000" xyz="-0.064000 0.000000 -0.000500"/>
-      <geometry>
-        <mesh filename="$(arg mesh_uri)/storage_collision/storage_7.stl" scale="0.001 0.001 0.001"/>
-      </geometry>
-    </collision>
-    <collision name="storage_collision_8">
-      <origin rpy="1.570796 0.000000 0.000000" xyz="-0.064000 0.000000 -0.000500"/>
-      <geometry>
-        <mesh filename="$(arg mesh_uri)/storage_collision/storage_8.stl" scale="0.001 0.001 0.001"/>
+        <sphere radius="0.004763" />
       </geometry>
     </collision>
   </link>
   <joint name="wheel_left_joint" type="continuous">
-    <parent link="base_link"/>
-    <child link="wheel_left_link"/>
-    <origin rpy="0.000000 -0.000000 0.000000" xyz="0.000000 0.143900 0.023000"/>
-    <axis xyz="0 1 0"/>
-    <limit effort="3.0" velocity="8.063"/>
+    <parent link="base_link" />
+    <child link="wheel_left_link" />
+    <origin rpy="0.000000 -0.000000 0.000000" xyz="0.000000 0.143900 0.023000" />
+    <axis xyz="0 1 0" />
+    <limit effort="3.0" velocity="8.063" />
   </joint>
   <link name="wheel_left_link">
     <inertial>
-      <origin rpy="0 0 0" xyz="0.000000 -0.000704 0.000002"/>
-      <mass value="0.028500"/>
-      <inertia ixx="1.1098e-05" ixy="5.7318e-09" ixz="3.1818e-09" iyy="2.0549e-05" iyz="-4.8114e-11" izz="1.1095e-05"/>
+      <origin rpy="0 0 0" xyz="0.000000 -0.000704 0.000002" />
+      <mass value="0.028500" />
+      <inertia ixx="1.1098e-05" ixy="5.7318e-09" ixz="3.1818e-09" iyy="2.0549e-05" iyz="-4.8114e-11" izz="1.1095e-05" />
     </inertial>
     <visual>
-      <origin rpy="0 0 0" xyz="0 0 0"/>
+      <origin rpy="0 0 0" xyz="0 0 0" />
       <geometry>
-        <mesh filename="$(arg mesh_uri)/wheel_left_link.stl" scale="0.001 0.001 0.001"/>
+        <mesh filename="$(arg mesh_uri)/wheel_left_link.stl" scale="0.001 0.001 0.001" />
       </geometry>
     </visual>
     <collision>
-      <origin rpy="1.570796 0 0" xyz="0 0 0"/>
+      <origin rpy="1.570796 0 0" xyz="0 0 0" />
       <geometry>
-        <cylinder length="0.015000" radius="0.033000"/>
+        <cylinder length="0.015000" radius="0.033000" />
       </geometry>
     </collision>
   </link>
   <joint name="wheel_right_joint" type="continuous">
-    <parent link="base_link"/>
-    <child link="wheel_right_link"/>
-    <origin rpy="0.000000 -0.000000 0.000000" xyz="0.000000 -0.143900 0.023000"/>
-    <axis xyz="0 1 0"/>
-    <limit effort="3.0" velocity="8.063"/>
+    <parent link="base_link" />
+    <child link="wheel_right_link" />
+    <origin rpy="0.000000 -0.000000 0.000000" xyz="0.000000 -0.143900 0.023000" />
+    <axis xyz="0 1 0" />
+    <limit effort="3.0" velocity="8.063" />
   </joint>
   <link name="wheel_right_link">
     <inertial>
-      <origin rpy="0 0 0" xyz="0.000000 0.000704 -0.000002"/>
-      <mass value="0.028500"/>
-      <inertia ixx="1.1098e-05" ixy="-5.7318e-09" ixz="-3.1818e-09" iyy="2.0549e-05" iyz="-4.8114e-11" izz="1.1095e-05"/>
+      <origin rpy="0 0 0" xyz="0.000000 0.000704 -0.000002" />
+      <mass value="0.028500" />
+      <inertia ixx="1.1098e-05" ixy="-5.7318e-09" ixz="-3.1818e-09" iyy="2.0549e-05" iyz="-4.8114e-11" izz="1.1095e-05" />
     </inertial>
     <visual>
-      <origin rpy="0 0 0" xyz="0 0 0"/>
+      <origin rpy="0 0 0" xyz="0 0 0" />
       <geometry>
-        <mesh filename="$(arg mesh_uri)/wheel_right_link.stl" scale="0.001 0.001 0.001"/>
+        <mesh filename="$(arg mesh_uri)/wheel_right_link.stl" scale="0.001 0.001 0.001" />
       </geometry>
     </visual>
     <collision>
-      <origin rpy="1.570796 0 0" xyz="0 0 0"/>
+      <origin rpy="1.570796 0 0" xyz="0 0 0" />
       <geometry>
-        <cylinder length="0.015000" radius="0.033000"/>
+        <cylinder length="0.015000" radius="0.033000" />
       </geometry>
     </collision>
   </link>
-  <joint name="pole_front_cam_joint" type="fixed">
-    <parent link="base_link"/>
-    <child link="pole_front_cam_link"/>
-    <origin rpy="0.000000 0.314159 0.000000" xyz="-0.137869 0.000185 0.434932"/>
+  <link name="imu_link" />
+  <joint name="imu_joint" type="fixed">
+    <parent link="base_link" />
+    <child link="imu_link" />
+    <origin rpy="0 0 0" xyz="0.0178 0 0.0585" />
+    <!-- x: waffle front edge 0.0688 - 0.051 (measured); z: OpenCR board top in base_link mesh -->
   </joint>
-  <link name="pole_front_cam_link">
-    <inertial>
-      <origin rpy="0 0 0" xyz="-0.013393 0.001408 -0.000023"/>
-      <mass value="0.072000"/>
-      <inertia ixx="4.6203e-05" ixy="4.1597e-07" ixz="2.0009e-08" iyy="6.9218e-06" iyz="3.6648e-09" izz="4.6614e-05"/>
-    </inertial>
+  <!-- basket slots: cell floor center, 3 rows (x, pole -> arm) x 4 cols (y, -y -> +y) -->
+  <!-- ================= ros2_control ================= -->
+  <!-- LDS-03 라이다: 1층 맨 앞, 두 바퀴 사이 가운데 (x·z는 실측 전 — tb3_bringup URDF lidar_x/lidar_z와 같게) -->
+  <joint name="scan_joint" type="fixed">
+    <parent link="base_link" />
+    <child link="base_scan" />
+    <origin rpy="0 0 0" xyz="0.060 0 0.022" />
+  </joint>
+  <link name="base_scan">
     <visual>
-      <origin rpy="0 0 0" xyz="0 0 0"/>
       <geometry>
-        <mesh filename="$(arg mesh_uri)/camera_rear_link.stl" scale="0.001 0.001 0.001"/>
+        <box size="0.0397 0.0547 0.034" />
       </geometry>
     </visual>
     <collision>
-      <origin rpy="0.000000 0.000000 0.000000" xyz="-0.012525 -0.000058 -0.000000"/>
       <geometry>
-        <box size="0.025050 0.089714 0.025000"/>
+        <box size="0.0397 0.0547 0.034" />
       </geometry>
     </collision>
   </link>
-  <joint name="arm_mount_joint" type="fixed">
-    <parent link="base_link"/>
-    <child link="arm_base_link"/>
-    <origin rpy="-0.000000 0.000000 0.000000" xyz="0.047985 -0.00023 0.130175"/>
-  </joint>
-  <link name="arm_base_link">
-    <inertial>
-      <origin rpy="0.0 0.0 0.0" xyz="-0.01169226743052282 -3.774353380840405e-15 0.023926534323405226"/>
-      <mass value="0.08108257974970318"/>
-      <inertia ixx="1.2862502962900217e-05" ixy="6.251056457349735e-19" ixz="-1.811662342359175e-07" iyy="2.2531969968508323e-05" iyz="1.5086560978736273e-17" izz="1.9821050957242446e-05"/>
-    </inertial>
-    <visual name="arm_base_link_visual">
-      <origin rpy="0.0 -0.0 0.0" xyz="0.0 0.0 0.0"/>
-      <geometry>
-        <mesh filename="$(arg mesh_uri)/arm_base_1.stl" scale="0.001 0.001 0.001"/>
-      </geometry>
-    </visual>
-    <collision name="arm_base_link_collision">
-      <origin rpy="0.0 -0.0 0.0" xyz="0.0 0.0 0.0"/>
-      <geometry>
-        <mesh filename="$(arg mesh_uri)/arm_base_1.stl" scale="0.001 0.001 0.001"/>
-      </geometry>
-    </collision>
-  </link>
-  <link name="shoulder_link">
-    <inertial>
-      <origin rpy="0.0 0.0 0.0" xyz="0.0 0.000668578344313189 0.028869490461060965"/>
-      <mass value="0.08583374201044289"/>
-      <inertia ixx="2.6324742259425243e-05" ixy="-7.312006911381859e-16" ixz="-9.128905585988183e-18" iyy="2.2861624315008813e-05" iyz="-8.980408739570743e-08" izz="1.4187591495603722e-05"/>
-    </inertial>
-    <visual name="shoulder_link_visual">
-      <origin rpy="0.0 0.0 0.0" xyz="0.0 0.0 -0.0409"/>
-      <geometry>
-        <mesh filename="$(arg mesh_uri)/shoulder_1.stl" scale="0.001 0.001 0.001"/>
-      </geometry>
-    </visual>
-    <collision name="shoulder_link_collision">
-      <origin rpy="0.0 0.0 0.0" xyz="0.0 0.0 -0.0409"/>
-      <geometry>
-        <mesh filename="$(arg mesh_uri)/shoulder_1.stl" scale="0.001 0.001 0.001"/>
-      </geometry>
-    </collision>
-  </link>
-  <link name="upper_arm_link">
-    <inertial>
-      <origin rpy="1.570796326794511 0.0 3.141592653375372" xyz="0.008487065078161757 0.0004453244413869725 0.10499673065502808"/>
-      <mass value="0.12886465633856012"/>
-      <inertia ixx="0.00018774476358412258" ixy="2.3927185167595554e-05" ixz="2.494779573069466e-07" iyy="3.578068745086586e-05" iyz="-1.3200789827030247e-06" izz="0.00019584173585813564"/>
-    </inertial>
-    <visual name="upper_arm_link_visual">
-      <origin rpy="0.0 0.0 0.0" xyz="0.0 0.0 -0.08249999999999999"/>
-      <geometry>
-        <mesh filename="$(arg mesh_uri)/link1_1.stl" scale="0.001 0.001 0.001"/>
-      </geometry>
-    </visual>
-    <collision name="upper_arm_link_collision">
-      <origin rpy="0.0 0.0 0.0" xyz="0.0 0.0 -0.08249999999999999"/>
-      <geometry>
-        <mesh filename="$(arg mesh_uri)/link1_1.stl" scale="0.001 0.001 0.001"/>
-      </geometry>
-    </collision>
-  </link>
-  <link name="forearm_link">
-    <inertial>
-      <origin rpy="1.5707963267949108 0.0 3.14159265337551" xyz="0.0937959598859132 0.0004892301406918195 6.576999200189225e-07"/>
-      <mass value="0.117299760592073"/>
-      <inertia ixx="1.9524545623177503e-05" ixy="-2.9158900918577e-09" ixz="1.0925502645848908e-06" iyy="0.00014316575812332259" iyz="3.773501040795638e-11" izz="0.00013706538722077516"/>
-    </inertial>
-    <visual name="forearm_link_visual">
-      <origin rpy="0.0 0.0 0.0" xyz="-0.023999999999999997 0.0 -0.21050000000000005"/>
-      <geometry>
-        <mesh filename="$(arg mesh_uri)/link2_1.stl" scale="0.001 0.001 0.001"/>
-      </geometry>
-    </visual>
-    <collision name="forearm_link_collision">
-      <origin rpy="0.0 0.0 0.0" xyz="-0.023999999999999997 0.0 -0.21050000000000005"/>
-      <geometry>
-        <mesh filename="$(arg mesh_uri)/link2_1.stl" scale="0.001 0.001 0.001"/>
-      </geometry>
-    </collision>
-  </link>
-  <link name="wrist_link">
-    <inertial>
-      <origin rpy="1.570796326794886 0.0 3.1415926533755343" xyz="0.04362261925352582 -4.4208071231510715e-11 0.01144891623665953"/>
-      <mass value="0.09015230299876778"/>
-      <inertia ixx="2.376831067770098e-05" ixy="5.954218246732174e-07" ixz="-3.5110061152839838e-15" iyy="1.98868978503507e-05" iyz="2.3069523907684884e-16" izz="2.9205178935103743e-05"/>
-    </inertial>
-    <visual name="wrist_link_visual">
-      <origin rpy="0.0 0.0 0.0" xyz="-0.148 0.0 -0.2105"/>
-      <geometry>
-        <mesh filename="$(arg mesh_uri)/wrist_1.stl" scale="0.001 0.001 0.001"/>
-      </geometry>
-    </visual>
-    <collision name="wrist_link_collision">
-      <origin rpy="0.0 0.0 0.0" xyz="-0.148 0.0 -0.2105"/>
-      <geometry>
-        <mesh filename="$(arg mesh_uri)/wrist_1.stl" scale="0.001 0.001 0.001"/>
-      </geometry>
-    </collision>
-  </link>
-  <link name="gripper_link">
-    <inertial>
-      <origin rpy="-1.5707963267948966 0.0 -1.5707963270091663" xyz="0.03333120209251042 1.5886189045943526e-07 0.008076961447025329"/>
-      <mass value="0.17574131271191906"/>
-      <inertia ixx="7.566997046639816e-05" ixy="4.58037525130514e-08" ixz="1.147686837904163e-09" iyy="0.00010679192530828156" iyz="-8.666284099644634e-06" izz="0.00010974001130350429"/>
-    </inertial>
-    <visual name="gripper_link_visual">
-      <origin rpy="0.0 0.0 -4.2852856514244266e-10" xyz="-0.21089999999999998 0.0 -0.21050000000000005"/>
-      <geometry>
-        <mesh filename="$(arg mesh_uri)/gripper_body_1.stl" scale="0.001 0.001 0.001"/>
-      </geometry>
-    </visual>
-    <collision name="gripper_link_collision">
-      <origin rpy="0.0 0.0 -4.2852856514244266e-10" xyz="-0.21089999999999998 0.0 -0.21050000000000005"/>
-      <geometry>
-        <mesh filename="$(arg mesh_uri)/gripper_body_1.stl" scale="0.001 0.001 0.001"/>
-      </geometry>
-    </collision>
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