Commit message: isaac: 개념 실습 L1~L3를 steps/로 통합, L3 IMU+LiDAR (실제 USD prim 경로)

File: isaac/urdf/beebot/urdf.xacro (robot description, xacro)
@@ -82,4 +82,10 @@
     <link name="caster_back_${side}_link">
       <collision><geometry><sphere radius="0.004763"/></geometry></collision>
+      <!-- 센서(IMU/RayCaster) rigid body view가 zero-mass 링크에서 깨지지 않게 작은 관성 추가.
+           실제 캐스터 볼+마운트 ~5 g, 구 관성 2/5·m·r² ≈ 9e-8 -->
+      <inertial>
+        <mass value="0.005"/>
+        <inertia ixx="1e-7" ixy="0" ixz="0" iyy="1e-7" iyz="0" izz="1e-7"/>
+      </inertial>
     </link>
   </xacro:macro>
